Commit message: Update dyxel_arm_description.urdf
There was a mistake in the limit part of the urdf file. I fixed it.

File: urdf/dyxel_arm_description.urdf (robot description, URDF)
Before this commit: robot dyxel_arm_description, 8 links, 7 joints
Joints:
- joint joint_1: limit lower=0 upper=0 effort=0 velocity=0 -> lower=-3.14 upper=3.14 effort=100 velocity=0.5
- joint joint_2: limit lower=0 upper=0 effort=0 velocity=0 -> lower=-3.14 upper=3.14 effort=100 velocity=0.5
- joint joint_3: limit lower=0 upper=0 effort=0 velocity=0 -> lower=-3.14 upper=3.14 effort=100 velocity=0.5
- joint joint_4: limit lower=0 upper=0 effort=0 velocity=0 -> lower=-3.14 upper=3.14 effort=100 velocity=0.5
- joint joint_5: limit lower=0 upper=0 effort=0 velocity=0 -> lower=-3.14 upper=3.14 effort=100 velocity=0.5
- joint joint_6: limit lower=0 upper=0 effort=0 velocity=0 -> lower=-3.14 upper=3.14 effort=100 velocity=0.5
- joint joint_7: limit lower=0 upper=0 effort=0 velocity=0 -> lower=-3.14 upper=3.14 effort=100 velocity=0.5
